Commit message: Remove world link and world joint from URDF/XACRO

File: model/URDF/walking_robot.urdf (robot description, URDF)
Before this commit: robot walking_robot, 14 links, 13 joints
Links:
- removed link world
Joints:
- removed joint world_jt

File: model/URDF/walking_robot.xacro (robot description, xacro)
@@ -86,5 +86,5 @@
 <!--////////////////////////////////////////////////////////ROBOT DEFINITION\\\\\\\\\\\\\\\\\\\\\\\\\\\\\\\\\\\\\\\\\\\\\\\\\\\\\-->
 <!--World-->
-	<link name="world" />
+<!--	<link name="world" />-->
 <!--Robot base-->
 	<link name="walker_base">
@@ -102,8 +102,8 @@
 	<xacro:leg name="HL" color="${light_red}" r1="-1" r2="-1"/>
 	<xacro:leg name="HR" color="${light_red}" r1="1" r2="-1"/>
-	<joint name="world_jt" type="floating">
-		<parent link="world"/>
-		<child link="walker_base"/>
-	</joint>
+<!--	<joint name="world_jt" type="floating">-->
+<!--		<parent link="world"/>-->
+<!--		<child link="walker_base"/>-->
+<!--	</joint>-->
 	<xacro:joint_mac leg_name="FL" number="1" parent_="walker_base" child_="link_1_FL" r1="-1" r2="1" />
 	<xacro:joint_mac leg_name="FL" number="2" parent_="link_1_FL" child_="link_2_FL" r1="-1" r2="1" />

Commit message: Update URDF description of the robot

File: model/URDF/walking_robot.urdf (robot description, URDF)
Before this commit: robot walking_robot, 13 links, 12 joints
Links:
- added link tip_FL; collision sphere radius=0.03; visual sphere radius=0.03
- added link tip_FR; collision sphere radius=0.03; visual sphere radius=0.03
- added link tip_HL; collision sphere radius=0.03; visual sphere radius=0.03
- added link tip_HR; collision sphere radius=0.03; visual sphere radius=0.03
Joints:
- added joint FL_tip_joint: type fixed, parent link_3_FL, child tip_FL, origin xyz=0 0.3 0
- added joint FR_tip_joint: type fixed, parent link_3_FR, child tip_FR, origin xyz=0 0.3 0
- added joint HL_tip_joint: type fixed, parent link_3_HL, child tip_HL, origin xyz=0 -0.3 0
- added joint HR_tip_joint: type fixed, parent link_3_HR, child tip_HR, origin xyz=0 -0.3 0

File: model/URDF/walking_robot.xacro (robot description, xacro)
@@ -59,4 +59,20 @@
 		</link>
 	</xacro:macro>
+	<!-- Leg Tip Macro -->
+	<xacro:macro name="leg_tip" params="leg_name">
+		<link name="tip_${leg_name}">
+			<visual>
+				<geometry>
+					<sphere radius="${tip_radius}" />
+				</geometry>
+				<material name="mat_${leg_name}" />
+			</visual>
+			<collision>
+				<geometry>
+					<sphere radius="${tip_radius}" />
+				</geometry>
+			</collision>
+		</link>
+	</xacro:macro>
 	<!--Leg Macro-->
 	<xacro:macro name="leg" params="name color r1 r2">
@@ -84,4 +100,12 @@
 		</joint>
 	</xacro:macro>
+	<!-- Fixed Joint Macro -->
+	<xacro:macro name="tip_jt" params="leg_name r2">
+		<joint name="${leg_name}_tip_joint" type="fixed">
+			<parent link="link_3_${leg_name}" />
+			<child link="tip_${leg_name}" />
+			<origin xyz="0 ${r2*link_3_length} 0"/>
+		</joint>
+	</xacro:macro>
 <!--////////////////////////////////////////////////////////ROBOT DEFINITION\\\\\\\\\\\\\\\\\\\\\\\\\\\\\\\\\\\\\\\\\\\\\\\\\\\\\-->
 <!--World-->
@@ -102,4 +126,8 @@
 	<xacro:leg name="HL" color="${light_red}" r1="-1" r2="-1"/>
 	<xacro:leg name="HR" color="${light_red}" r1="1" r2="-1"/>
+	<xacro:leg_tip leg_name="FL" />
+	<xacro:leg_tip leg_name="FR" />
+	<xacro:leg_tip leg_name="HL" />
+	<xacro:leg_tip leg_name="HR" />
 <!--	<joint name="world_jt" type="floating">-->
 <!--		<parent link="world"/>-->
@@ -118,3 +146,7 @@
 	<xacro:joint_mac leg_name="HR" number="2" parent_="link_1_HR" child_="link_2_HR" r1="1" r2="-1" />
 	<xacro:joint_mac leg_name="HR" number="3" parent_="link_2_HR" child_="link_3_HR" r1="1" r2="-1" />
+	<xacro:tip_jt leg_name="FL" r2="1" />
+	<xacro:tip_jt leg_name="FR" r2="1" />
+	<xacro:tip_jt leg_name="HL" r2="-1" />
+	<xacro:tip_jt leg_name="HR" r2="-1" />
 </robot>
